File: indicator/scheme/indicator.kicad_pcb (KiCad board)
At the start: 2 copper layers, 52 x 54.5 mm, 51 parts, among them J1 Amplifier, SW1 mode, U1 LM3915, U2 LM3915

Commit message: small: QR code
Change QR code from github to site.
Parts:
- removed the G*** at (130.0, 98.2)
- added G***: LOGO, mine:qr_code, B.Cu at (130.0, 98.0)
